File: STM32.kicad_pcb (KiCad board)
At the start: 2 copper layers, 41 x 31 mm, 32 parts, among them J1 Conn_01x04_Male, J2 Conn_01x04_Male, J3 Conn_01x04_Male, J4 USB_B_Micro, SW1 SW_SPDT, U1 AMS1117-3.3, U2 STM32F103C8T6, Y1 16MHz

Commit message: traced some here and there
Parts:
- moved R3 3.73 mm to (116.2, 87.0)
- moved R2 3.64 mm to (113.8, 86.9)
- moved J1 1.50 mm to (114.8, 64.0)
- moved J3 1.00 mm to (129.8, 64.0)
- moved J2 0.89 mm to (110.8, 90.7)
- moved C7 0.70 mm to (118.7, 83.6)
- moved C12 0.36 mm to (109.2, 82.1)
- moved R4 0.27 mm to (103.1, 72.7)
- moved C13 0.27 mm to (109.2, 83.4)
- moved R5 0.16 mm to (125.4, 75.5)
- moved C4 0.15 mm to (113.5, 83.6)
- moved FB1 0.15 mm to (111.0, 82.8)
- moved J4 0.09 mm to (133.9, 76.0)
Routing:
- net /BOOT0: track 0.00 -> 20.3 mm
- net /SWDIO: track 0.00 -> 16.1 mm
- net /USART1_RX: track 0.00 -> 15.1 mm
- net /USART1_TX: track 0.00 -> 13.8 mm
- net GND: track 7.51 -> 20.0 mm, vias 0 -> 10
- net /USB_D+: track 0.00 -> 12.2 mm
- net /USB_D-: track 0.00 -> 12.1 mm
- net /SWCLK: track 0.00 -> 11.8 mm
- net /I2C2_SCL: track 0.00 -> 11.1 mm
- net /I2C2_SDA: track 0.00 -> 9.74 mm
- net /NRST: track 0.00 -> 8.97 mm
- net /HSE_IN: track 0.00 -> 7.73 mm
- net /HSE_OUT: track 0.00 -> 5.59 mm
- net +3.3V: track 7.41 -> 9.67 mm
- net /SW_BOOT0: track 0.28 -> 2.54 mm

Commit message: nothing much
Routing:
- net GND: track 20.0 -> 22.7 mm, vias 10 -> 18
Changed lines of the file:
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@@
 		(tags "capacitor")
 		(property "Reference" "C9"
-			(at 0 -1.5 180)
+			(at -1.640293 0.000826 180)
 			(layer "F.SilkS")
 			(effects
@@
 	)
 	(segment
-		(start 121.316521 75.433479)
-		(end 121.878632 75.433479)
+		(start 121.878632 75.433479)
+		(end 122.715015 75.433479)
+		(width 0.3)
+		(layer "F.Cu")
+		(net "GND")
+	)
+	(segment
+		(start 120.95873 75.20873)
+		(end 121.183479 75.433479)
 		(width 0.3)
 		(layer "F.Cu")
@@
 	)
 	(segment
+		(start 119.936707 75.20873)
+		(end 120.95873 75.20873)
+		(width 0.3)
+		(layer "F.Cu")
+		(net "GND")
+	)
+	(segment
 		(start 118.024207 83.433591)
 		(end 118.210109 83.619493)
@@
 	)
 	(segment
-		(start 119.936707 75.20873)
-		(end 120.95873 75.20873)
-		(width 0.3)
-		(layer "F.Cu")
-		(net "GND")
-	)
-	(segment
 		(start 108.749849 82.086434)
 		(end 108.749849 81.267084)
@@
 	)
 	(segment
+		(start 135.183559 81.948772)
+		(end 135.187765 81.952978)
+		(width 0.5)
+		(layer "F.Cu")
+		(net "GND")
+	)
+	(segment
 		(start 110.70873 78.20873)
 		(end 110.5 78)
@@
 	)
 	(segment
+		(start 121.183479 75.433479)
+		(end 121.878632 75.433479)
+		(width 0.3)
+		(layer "F.Cu")
+		(net "GND")
+	)
+	(segment
 		(start 113.524207 73.29623)
 		(end 113.524207 72.45561)
@@
 	)
 	(segment
-		(start 120.95873 75.20873)
-		(end 121.25 75.5)
-		(width 0.3)
-		(layer "F.Cu")
-		(net "GND")
-	)
-	(segment
 		(start 113.524207 72.45561)
 		(end 113.739909 72.239908)
@@
 	)
 	(segment
-		(start 121.25 75.5)
-		(end 121.316521 75.433479)
-		(width 0.3)
-		(layer "F.Cu")
-		(net "GND")
-	)
-	(segment
 		(start 108.61 77.017313)
 		(end 109 76.627313)
@@
 	)
 	(segment
+		(start 122.715015 75.433479)
+		(end 122.722222 75.440686)
+		(width 0.3)
+		(layer "F.Cu")
+		(net "GND")
+	)
+	(segment
 		(start 113.739909 72.239908)
 		(end 113.73 72.229999)
@@
 	)
 	(segment
+		(start 130.998993 74.732094)
+		(end 130.990942 74.724043)
+		(width 0.3)
+		(layer "F.Cu")
+		(net "GND")
+	)
+	(segment
 		(start 114.002814 83.635378)
 		(end 114.411486 83.635378)
@@
 	)
 	(segment
+		(start 132.049957 74.732094)
+		(end 130.998993 74.732094)
+		(width 0.3)
+		(layer "F.Cu")
+		(net "GND")
+	)
+	(segment
 		(start 118.024207 81.62123)
 		(end 118.024207 83.433591)
@@
 		(net "GND")
 	)
+	(segment
+		(start 134.352924 81.948772)
+		(end 135.183559 81.948772)
+		(width 0.5)
+		(layer "F.Cu")
+		(net "GND")
+	)
 	(via
 		(at 108.719838 84.263484)
@@
 	)
 	(via
+		(at 127.5 79.5)
+		(size 0.6)
+		(drill 0.3)
+		(layers "F.Cu" "B.Cu")
+		(net "GND")
+	)
+	(via
+		(at 127.5 78.5)
+		(size 0.6)
+		(drill 0.3)
+		(layers "F.Cu" "B.Cu")
+		(net "GND")
+	)
+	(via
 		(at 109.766972 72.843349)
 		(size 0.7)
@@
 	)
 	(via
+		(at 127.297926 82.683681)
+		(size 0.6)
+		(drill 0.3)
+		(layers "F.Cu" "B.Cu")
+		(net "GND")
+	)
+	(via
+		(at 130.990942 74.724043)
+		(size 0.6)
+		(drill 0.3)
+		(layers "F.Cu" "B.Cu")
+		(net "GND")
+	)
+	(via
+		(at 128.144037 82.68964)
+		(size 0.6)
+		(drill 0.3)
+		(layers "F.Cu" "B.Cu")
+		(net "GND")
+	)
+	(via
 		(at 108.154801 74.178177)
 		(size 0.6)
@@
 	)
 	(via
+		(at 122.722222 75.440686)
+		(size 0.6)
+		(drill 0.3)
+		(layers "F.Cu" "B.Cu")
+		(net "GND")
+	)
+	(via
 		(at 118.040023 80.326566)
 		(size 0.6)
@@
 	)
 	(via
+		(at 131.312007 83.140993)
+		(size 0.6)
+		(drill 0.3)
+		(layers "F.Cu" "B.Cu")
+		(net "GND")
+	)
+	(via
 		(at 109 76.627313)
 		(size 0.6)
 		(drill 0.3)
+		(layers "F.Cu" "B.Cu")
+		(net "GND")
+	)
+	(via
+		(at 135.187765 81.952978)
+		(size 0.6)
+		(drill 0.3)

Commit message: forgot the manufacturing files
Parts:
- moved R4 1.45 mm to (103.0, 71.2)
- moved C13 0.15 mm to (109.2, 83.6)
- moved R5 0.09 mm to (125.3, 75.5)
- moved C12 0.09 mm to (109.2, 82.0)
Routing:
- net +3.3V: track 9.67 -> 156.9 mm, vias 0 -> 6
- net +3.3VA: track 1.97 -> 6.29 mm
- net GND: track 22.7 -> 25.2 mm, vias 18 -> 20
- net /PWR_LED_K: track 0.00 -> 1.59 mm
- net /BOOT0: track 20.3 -> 18.9 mm
- net /SW_BOOT0: track 2.54 -> 3.81 mm
- added copper zone on F.Cu, net +3.3V
- added copper zone on F.Cu, net GND
- added copper zone on F.Cu, net VBUS
Other:
- board text added: "BOOT"
- board text added: "I2C"
- board text added: "ON"
- board text added: "SWD"
- board text added: "UART"
- board text added: "USB"
