File: STM32.kicad_sch (KiCad schematic)
At the start: 32 parts, among them J1 Conn_01x04_Male, J2 Conn_01x04_Male, J3 Conn_01x04_Male, J4 USB_B_Micro, SW1 SW_SPDT, U1 AMS1117-3.3, U2 STM32F103C8T6, Y1 16MHz

Commit message: forgot the manufacturing files
Parts:
- C1, C2: LCSC (none) -> C45783
- C10, C4, C6, C7, C9: LCSC (none) -> C1525
- C11: LCSC (none) -> C15195
- C12, C13: LCSC (none) -> C52923
- C3: LCSC (none) -> C19702
- C5, C8: LCSC (none) -> C32949
- D1: LCSC (none) -> C2286
- R1, R2, R3, R5: LCSC (none) -> C25867
- R4: LCSC (none) -> C25744
- SW1: LCSC (none) -> C221841
- U1: LCSC (none) -> C6186
- U2: LCSC (none) -> C8734
- Y1: LCSC (none) -> C13738
